File: right-pcb/row_staggered_split_keyboard_right_side.kicad_pcb (KiCad board)
At the start: 2 copper layers, 165 x 132 mm, 177 parts, among them J1 Conn_01x02, SW1 SW_SPST, SW10 SW_SPST, SW11 SW_SPST, SW12 SW_SPST, SW13 SW_SPST, SW14 SW_SPST, SW15 SW_SPST, SW16 SW_SPST, SW17 SW_SPST, SW18 SW_SPST, SW19 SW_SPST, SW2 SW_SPST, SW20 SW_SPST, SW21 SW_SPST, SW22 SW_SPST, SW23 SW_SPST, SW24 SW_SPST, SW25 SW_SPST, SW26 SW_SPST, SW27 SW_SPST, SW28 SW_SPST, SW29 SW_SPST, SW3 SW_SPST, SW30 SW_SPST, SW31 SW_SPST, SW32 SW_SPST, SW33 SW_SPST, SW34 SW_SPST, SW35 SW_SPST, SW36 SW_SPST, SW37 SW_SPST, SW38 SW_SPST, SW39 SW_SPST, SW4 SW_SPST, SW40 SW_SPST, SW41 SW_SPST, SW5 SW_SPST, SW6 SW_SPST, SW7 SW_SPST, SW8 SW_SPST, SW9 SW_SPST, U1 SN74LVC1T45DBV

Commit message: applied feedback from coworker
Parts:
- moved C1 1.01 mm to (173.8, 45.0)
- moved C4 0.86 mm to (160.9, 44.5)
Routing:
- net /R1C5/DOUT: track 102.2 -> 104.2 mm
- net GND: track 166.2 -> 168.1 mm
- net +3V3: track 4.96 -> 5.97 mm
- net +5V: track 4.28 -> 5.14 mm
- added copper zone on B.Cu, net GND

Commit message: adding mounting hole in center for additional support, and cleaning up tracks/zones
Parts:
- added H5: M2, MountingHole:MountingHole_2.2mm_M2, F.Cu at (108.2, 96.3)
- renumbered C12 to C11, C13 to C12, C14 to C13, C15 to C14, C16 to C15, C17 to C16, C18 to C17, C19 to C18, C20 to C19, C21 to C20, C22 to C21, C23 to C22, C24 to C23, C25 to C24, C11 to C25, D15 to D13, D16 to D14, D17 to D15, D18 to D16, D19 to D17, D20 to D18, D21 to D19, D22 to D20, D23 to D21, D24 to D22, D25 to D23, D26 to D24, D27 to D25, D28 to D26, D29 to D27, D30 to D28, D31 to D29, D32 to D30, D33 to D31, D34 to D32, D35 to D33, D36 to D34, D37 to D35, D38 to D36, D39 to D37, D40 to D38, D41 to D39, D42 to D40, D13 to D41, D14 to D42, H5 to H6, H6 to H7, SW11 to SW10, SW12 to SW11, SW13 to SW12, SW14 to SW13, SW15 to SW14, SW16 to SW15, SW17 to SW16, SW18 to SW17, SW19 to SW18, SW20 to SW19, SW21 to SW20, SW7 to SW21, SW8 to SW7, SW9 to SW8, SW10 to SW9
Routing:
- net /ROW3: track 206.1 -> 208.4 mm
- net /ROW4: track 216.7 -> 218.8 mm
- net /ROW6: track 256.1 -> 257.5 mm
- net /ROW5: track 240.4 -> 241.7 mm
- removed copper zone on B.Cu, net GND
