File: right-pcb/switch_with_LED_2U25.kicad_sch (KiCad schematic)
At the start: 5 parts, among them SW31 SW_SPST

Commit message: initial placement of switches and modifications from left to right
Parts:
- renumbered C38 to C41, D61 to D73, D62 to D74, SW31 to SW37
Changed lines of the file:
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@@
 		(dnp no)
 		(fields_autoplaced yes)
-		(property "Reference" "SW31"
+		(property "Reference" "SW37"
 			(at 121.92 92.7099 90)
 			(effects
@@
 				)
 				(path "/cf145565-22e2-4e5a-8a27-915862c57a1b/ceb25589-dab0-4ec4-bc76-eeaced9b67af"
-					(reference "SW7")
+					(reference "SW37")
 					(unit 1)
 				)
@@
 		(dnp no)
 		(fields_autoplaced yes)
-		(property "Reference" "D62"
+		(property "Reference" "D74"
 			(at 138.43 125.6598 0)
 			(effects
@@
 				)
 				(path "/cf145565-22e2-4e5a-8a27-915862c57a1b/ceb25589-dab0-4ec4-bc76-eeaced9b67af"
-					(reference "D14")
+					(reference "D74")
 					(unit 1)
 				)
@@
 		(dnp no)
 		(fields_autoplaced yes)
-		(property "Reference" "#PWR0150"
+		(property "Reference" "#PWR0162"
 			(at 107.95 125.73 0)
 			(effects
@@
 				(path "/cf145565-22e2-4e5a-8a27-915862c57a1b/7de27539-085a-429d-8cb1-9e38513b42e6"
 					(reference "#PWR0150")
+					(unit 1)
+				)
+				(path "/cf145565-22e2-4e5a-8a27-915862c57a1b/ceb25589-dab0-4ec4-bc76-eeaced9b67af"
+					(reference "#PWR0162")
 					(unit 1)
 				)
@@
 		(dnp no)
 		(fields_autoplaced yes)
-		(property "Reference" "C38"
+		(property "Reference" "C41"
 			(at 110.49 113.0362 0)
 			(effects
@@
 				(path "/cf145565-22e2-4e5a-8a27-915862c57a1b/7de27539-085a-429d-8cb1-9e38513b42e6"
 					(reference "C38")
+					(unit 1)
+				)
+				(path "/cf145565-22e2-4e5a-8a27-915862c57a1b/ceb25589-dab0-4ec4-bc76-eeaced9b67af"
+					(reference "C41")
 					(unit 1)
 				)
@@
 		(dnp no)
 		(fields_autoplaced yes)
-		(property "Reference" "D61"
+		(property "Reference" "D73"
 			(at 123.19 102.8699 90)
 			(effects
@@
 				)
 				(path "/cf145565-22e2-4e5a-8a27-915862c57a1b/ceb25589-dab0-4ec4-bc76-eeaced9b67af"
-					(reference "D13")
+					(reference "D73")
 					(unit 1)
 				)
@@
 		(dnp no)
 		(fields_autoplaced yes)
-		(property "Reference" "#PWR0149"
+		(property "Reference" "#PWR0161"
 			(at 107.95 113.03 0)
 			(effects
@@
 				(path "/cf145565-22e2-4e5a-8a27-915862c57a1b/7de27539-085a-429d-8cb1-9e38513b42e6"
 					(reference "#PWR0149")
+					(unit 1)
+				)
+				(path "/cf145565-22e2-4e5a-8a27-915862c57a1b/ceb25589-dab0-4ec4-bc76-eeaced9b67af"
+					(reference "#PWR0161")
 					(unit 1)
 				)
@@
 		(dnp no)
 		(fields_autoplaced yes)
-		(property "Reference" "#PWR071"
+		(property "Reference" "#PWR0164"
 			(at 124.46 149.86 0)
 			(effects
@@
 				)
 				(path "/cf145565-22e2-4e5a-8a27-915862c57a1b/ceb25589-dab0-4ec4-bc76-eeaced9b67af"
-					(reference "#PWR023")
+					(reference "#PWR0164")
 					(unit 1)
 				)
@@
 					(unit 1)
 				)
+				(path "/cf145565-22e2-4e5a-8a27-915862c57a1b/ceb25589-dab0-4ec4-bc76-eeaced9b67af"
+					(reference "H6")
+					(unit 1)
+				)
 			)
 		)
@@
 		(dnp no)
 		(fields_autoplaced yes)
-		(property "Reference" "#PWR070"
+		(property "Reference" "#PWR0163"
 			(at 124.46 124.46 0)
 			(effects
@@
 				)
 				(path "/cf145565-22e2-4e5a-8a27-915862c57a1b/ceb25589-dab0-4ec4-bc76-eeaced9b67af"
-					(reference "#PWR022")
-					(unit 1)
-				)
+					(reference "#PWR0163")
+					(unit 1)
+				)

Commit message: adding mounting hole in center for additional support, and cleaning up tracks/zones
Parts:
- renumbered H6 to H7

Commit message: Boards were ordered
Parts:
- SW37: symbol Switch:SW_SPST -> SW-gElectroMech:SPST_MOM
Changed lines of the file:
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@@
 	)
 	(symbol
-		(lib_id "Switch:SW_SPST")
+		(lib_id "SW-gElectroMech:SPST_MOM")
 		(at 120.65 93.98 90)
 		(unit 1)
@@
 		)
 		(property "Datasheet" ""
-			(at 120.65 93.98 0)
+			(at 115.57 93.98 0)
 			(hide yes)
 			(show_name no)
@@
 			)
 		)
-		(property "Description" "Single Pole Single Throw (SPST) switch"
+		(property "Description" "Push button switch, generic, two pins"
 			(at 120.65 93.98 0)
 			(hide yes)
