File: left-pcb/switch_with_LED_2U25.kicad_sch (KiCad schematic)
At the start: 3 parts, among them SW28 SW_SPST

Commit message: Initial modifications to reduce fab cost and add caps
Removing 1 row and column of keys, and majorly changing layout

Routing still in progress
Parts:
- removed D55: D_Small, Diode_SMD:D_SOD-123, symbol Device:D_Small
- removed D56: SK6812MINI-E, SW-Adafruit:LED_SK6812MINI-E_REVERSE_MOUNT_3.2x2.8mm_P1.09mm, symbol SW-Adafruit:SK6812MINI-E
- removed SW28: SW_SPST, PCM_Switch_Keyboard_Hotswap_Kailh:SW_Hotswap_Kailh_MX_2.25u, symbol Switch:SW_SPST
- added C38: 100nF, Capacitor_SMD:C_1206_3216Metric_Pad1.33x1.80mm_HandSolder, symbol Device:C_Small
- added D67: D_Small, Diode_SMD:D_SOD-123, symbol Device:D_Small
- added D68: SK6812MINI-E, SW-Adafruit:LED_SK6812MINI-E_REVERSE_MOUNT_3.2x2.8mm_P1.09mm, symbol SW-Adafruit:SK6812MINI-E
- added SW34: SW_SPST, PCM_Switch_Keyboard_Hotswap_Kailh:SW_Hotswap_Kailh_MX_2.25u, symbol Switch:SW_SPST
Connections:
- net +5V: now also C38.1, D68.1 (VDD)
- net Column: now also D67.1 (K)
- net DIN: now also D68.4 (DIN)
- net DOUT: now also D68.2 (DOUT)
- net GND: now also C38.2, D68.3 (GND)
- net Row: now also SW34.2 (B)
- new net: D67.2 (A), SW34.1 (A)

Commit message: Caps, shrunk board, added mounting holes
Parts:
- C38: footprint Capacitor_SMD:C_1206_3216Metric_Pad1.33x1.80mm_HandSolder -> Capacitor_SMD:C_0805_2012Metric_Pad1.18x1.45mm_HandSolder
Changed lines of the file:
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@@
 			)
 		)
-		(property "Footprint" "Capacitor_SMD:C_1206_3216Metric_Pad1.33x1.80mm_HandSolder"
+		(property "Footprint" "Capacitor_SMD:C_0805_2012Metric_Pad1.18x1.45mm_HandSolder"
 			(at 107.95 114.3 0)
 			(effects

Commit message: Adding values to Diodes and adding stabilizers to 2U switches
Parts:
- D67: value D_Small -> 1N4148W
Changed lines of the file:
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@@
 			)
 		)
-		(property "Value" "D_Small"
+		(property "Value" "1N4148W"
 			(at 123.19 105.4099 90)
 			(effects

Commit message: Added extra column to left hand keyboard
Matching size to right hand side.
Parts:
- added H6: 2U Stabilizer, PCM_Mounting_Keyboard_Stabilizer:Stabilizer_Cherry_MX_2.00u, symbol Mechanical:MountingHole
Changed lines of the file:
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@@
 		(dnp no)
 		(fields_autoplaced yes)
-		(property "Reference" "#PWR0149"
+		(property "Reference" "#PWR0150"
 			(at 107.95 125.73 0)
 			(effects
@@
 			(project "row_staggered_split_keyboard_left_side"
 				(path "/cf145565-22e2-4e5a-8a27-915862c57a1b/72dbedf5-0b03-4be1-b418-6a53323f317d"
-					(reference "#PWR0149")
+					(reference "#PWR0150")
 					(unit 1)
 				)
@@
 		(dnp no)
 		(fields_autoplaced yes)
-		(property "Reference" "#PWR0148"
+		(property "Reference" "#PWR0149"
 			(at 107.95 113.03 0)
 			(effects
@@
 			(project "row_staggered_split_keyboard_left_side"
 				(path "/cf145565-22e2-4e5a-8a27-915862c57a1b/72dbedf5-0b03-4be1-b418-6a53323f317d"
-					(reference "#PWR0148")
+					(reference "#PWR0149")
 					(unit 1)
 				)
@@
 		(dnp no)
 		(fields_autoplaced yes)
-		(property "Reference" "#PWR0151"
+		(property "Reference" "#PWR0152"
 			(at 124.46 149.86 0)
 			(effects
@@
 				)
 				(path "/cf145565-22e2-4e5a-8a27-915862c57a1b/72dbedf5-0b03-4be1-b418-6a53323f317d"
-					(reference "#PWR0151")
+					(reference "#PWR0152")
 					(unit 1)
 				)
@@
 				(path "/cf145565-22e2-4e5a-8a27-915862c57a1b/febc083e-5fc3-4dde-a082-b48603250b8e"
 					(reference "#PWR075")
+					(unit 1)
+				)
+			)
+		)
+	)
+	(symbol
+		(lib_id "Mechanical:MountingHole")
+		(at 146.05 119.38 0)
+		(unit 1)
+		(exclude_from_sim no)
+		(in_bom yes)
+		(on_board yes)
+		(dnp no)
+		(fields_autoplaced yes)
+		(property "Reference" "H6"
+			(at 148.59 118.1099 0)
+			(effects
+				(font
+					(size 1.27 1.27)
+				)
+				(justify left)
+			)
+		)
+		(property "Value" "2U Stabilizer"
+			(at 148.59 120.6499 0)
+			(effects
+				(font
+					(size 1.27 1.27)
+				)
+				(justify left)
+			)
+		)
+		(property "Footprint" "PCM_Mounting_Keyboard_Stabilizer:Stabilizer_Cherry_MX_2.00u"
+			(at 146.05 119.38 0)
+			(effects
+				(font
+					(size 1.27 1.27)
+				)
+				(hide yes)
+			)
+		)
+		(property "Datasheet" "~"
+			(at 146.05 119.38 0)
+			(effects
+				(font
+					(size 1.27 1.27)
+				)
+				(hide yes)
+			)
+		)
+		(property "Description" "Mounting Hole without connection"
+			(at 146.05 119.38 0)
+			(effects
+				(font
+					(size 1.27 1.27)
+				)
+				(hide yes)
+			)
+		)
+		(instances
+			(project ""
+				(path "/cf145565-22e2-4e5a-8a27-915862c57a1b/72dbedf5-0b03-4be1-b418-6a53323f317d"
+					(reference "H6")
 					(unit 1)
 				)
@@
 		(dnp no)
 		(fields_autoplaced yes)
-		(property "Reference" "#PWR0150"
+		(property "Reference" "#PWR0151"
 			(at 124.46 124.46 0)
 			(effects
@@
 				)
 				(path "/cf145565-22e2-4e5a-8a27-915862c57a1b/72dbedf5-0b03-4be1-b418-6a53323f317d"
-					(reference "#PWR0150")
-					(unit 1)
-				)
+					(reference "#PWR0151")
+					(unit 1)
+				)

Commit message: adding mounting hole in center for additional support, and cleaning up tracks/zones
Parts:
- renumbered C38 to C44, D67 to D79, D68 to D80, H6 to H7, SW34 to SW40

Commit message: Boards were ordered
Parts:
- SW40: symbol Switch:SW_SPST -> SW-gElectroMech:SPST_MOM
Changed lines of the file:
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@@
 	)
 	(symbol
-		(lib_id "Switch:SW_SPST")
+		(lib_id "SW-gElectroMech:SPST_MOM")
 		(at 120.65 93.98 90)
 		(unit 1)
@@
 		)
 		(property "Datasheet" ""
-			(at 120.65 93.98 0)
+			(at 115.57 93.98 0)
 			(hide yes)
 			(show_name no)
@@
 			)
 		)
-		(property "Description" "Single Pole Single Throw (SPST) switch"
+		(property "Description" "Push button switch, generic, two pins"
 			(at 120.65 93.98 0)
 			(hide yes)
